Commit message: Update meshes name and xacros

File: mkmr_description/urdf/mkmr.xacro (robot description, xacro)
@@ -11,7 +11,13 @@
     <xacro:include filename="$(find mkmr_description)/urdf/common/plugins.gazebo.xacro"/>
     <xacro:include filename="$(find mkmr_description)/urdf/mkmr/mkmr_base.urdf.xacro"/>
+    <xacro:include filename="$(find mkmr_description)/urdf/mkmr/mkmr_wheels.urdf.xacro"/>
     <!-- <xacro:include filename="$(find mkmr_description)/urdf/sensors/rplidar_a1.urdf.xacro"/> -->
     <!-- Robot Base-->
     <xacro:mkmr_base/>
+     <!-- Wheels -->
+    <xacro:mkmr_wheels parent="${ROBOT_ID}/base_link" name="front_left_wheel" origin_xyz="0.35336 -0.30481 0.15788" origin_rpy="1.5708 0 -3.1416" axis="0 1 0"/>
+    <xacro:mkmr_wheels parent="${ROBOT_ID}/base_link" name="rear_left_wheel" origin_xyz="0.18836 -0.30481 0.15588" origin_rpy="-1.5708 0 0" axis="0 -1 0"/>
+    <xacro:mkmr_wheels parent="${ROBOT_ID}/base_link" name="front_right_wheel" origin_xyz="0.35336 -0.30481 -0.029122" origin_rpy="1.5708 0 -3.1416" axis="0 1 0"/>
+    <xacro:mkmr_wheels parent="${ROBOT_ID}/base_link" name="rear_right_wheel" origin_xyz="0.18836 -0.30481 -0.031122" origin_rpy="-1.5708 0 0" axis="0 -1 0"/>
     <!-- Laser -->
     <!-- <xacro:rplidar_a1 name="front_laser"

File: mkmr_description/urdf/mkmr/mkmr_base.urdf.xacro (robot description, xacro)
@@ -71,9 +71,41 @@
             </inertial>
         </link>
-        <joint name="${ROBOT_ID}/base_link_joint" type="fixed">
+        <joint name="${ROBOT_ID}/fMotor_joint" type="fixed">
             <origin xyz="0.30386 -0.34031 0.063378" rpy="1.5708 1.5708 0"/>
             <parent link="${ROBOT_ID}/base_link"/>
             <child link="${ROBOT_ID}/fMotor"/>
         </joint>
+        <!-- fDrivers -->
+        <link name="${ROBOT_ID}/fDrivers">
+            <visual>
+                <origin xyz="0 0 0" rpy="0 0 0"/>
+                <geometry>
+                    <mesh filename="package://mkmr_description/meshes/fDrivers.STL" />
+                </geometry>
+                <material name="Black"/>
+            </visual>
+            <collision>
+                <origin xyz="0 0 0" rpy="0 0 0"/>
+                <geometry>
+                    <mesh filename="package://mkmr_description/meshes/fDrivers.STL" />
+                </geometry>
+            </collision>
+            <inertial>
+                <origin xyz="-0.00660140608489862 0.0452390915749958 -0.00380039164943846"/>
+                <mass value="0.3"/>
+                <inertia
+                    ixx="9.00028132290921E-06"
+                    ixy="1.23322543868992E-07"
+                    ixz="1.33828527421449E-07"
+                    iyy="2.17066983097978E-05"
+                    iyz="7.70745731959558E-07"
+                    izz="2.83837538531001E-05" />
+            </inertial>
+        </link>
+        <joint name="${ROBOT_ID}/fDrivers_joint" type="fixed">
+            <origin xyz="0.26391 -0.33566 0.1011" rpy="-1.5708 0 -3.1416"/>
+            <parent link="${ROBOT_ID}/base_link"/>
+            <child link="${ROBOT_ID}/fDrivers"/>
+        </joint>
     </xacro:macro>
 </robot>
