Commit message: Update xacro files

File: mkmr_description/urdf/common/plugins.gazebo.xacro (robot description, xacro)
@@ -8,10 +8,4 @@
       <controlPeriod>0.002</controlPeriod>
     </plugin>
-    <!--plugin name="ground_truth" filename="libgazebo_ros_p3d.so">
-      <frameName>map</frameName>
-      <bodyName>base_footprint</bodyName>
-      <topicName>base_pose_ground_truth</topicName>
-      <updateRate>30.0</updateRate>
-    </plugin-->
   </gazebo>
 </robot>

File: mkmr_description/urdf/mkmr.xacro (robot description, xacro)
@@ -1,4 +1,5 @@
 <?xml version="1.0"?>
 <robot xmlns:xacro="http://ros.org/wiki/xacro" name="mkmr" >
+    <xacro:arg name="use_ros_control_for_base" default="true"/>
     <xacro:arg name="is_sim" default="false"/>
     <xacro:arg name="robot_id" default="mkmr0"/>
@@ -20,5 +21,7 @@
     <xacro:mkmr_wheels parent="${ROBOT_ID}/base_link" name="front_right_wheel" origin_xyz="0.35336 -0.30481 -0.029122" origin_rpy="1.5708 0 -3.1416" axis="0 1 0"/>
     <xacro:mkmr_wheels parent="${ROBOT_ID}/base_link" name="rear_right_wheel" origin_xyz="0.18836 -0.30481 -0.031122" origin_rpy="-1.5708 0 0" axis="0 -1 0"/>
+    <!-- <xacro:mkmr_wheels parent="${ROBOT_ID}/base_link" name="left_wheel_joint" origin_xyz="0.18836 -0.30481 0.15588" origin_rpy="-1.5708 0 0" axis="0 -1 0"/> -->
+    <!-- <xacro:mkmr_wheels parent="${ROBOT_ID}/base_link" name="right_wheel_joint" origin_xyz="0.35336 -0.30481 -0.029122" origin_rpy="1.5708 0 -3.1416" axis="0 1 0"/> -->
     <!-- Laser -->
-    <xacro:rplidar_a1 parent="${ROBOT_ID}/base_link" name="scan" origin_xyz="0.374625946277677 -0.494903544571783 0.0633776911630922" origin_rpy="0 0 3.14159265358979"/>
+    <!-- <xacro:rplidar_a1 parent="${ROBOT_ID}/base_link" name="scan" origin_xyz="0.374625946277677 -0.494903544571783 0.0633776911630922" origin_rpy="0 0 3.14159265358979"/> -->
 </robot>

File: mkmr_description/urdf/mkmr/mkmr_wheels.urdf.xacro (robot description, xacro)
@@ -6,5 +6,6 @@
                 <origin xyz="0 0 0" rpy="0 0 0"/>
                 <geometry>
-                    <mesh filename="package://mkmr_description/meshes/${name}.STL" />
+                    <!-- <mesh filename="package://mkmr_description/meshes/${name}.STL" /> -->
+                    <mesh filename="package://mkmr_description/meshes/front_left_wheel.STL" />
                 </geometry>
                 <material name="Black"/>
@@ -29,5 +30,5 @@
             </inertial>
         </link>
-        <joint name="${ROBOT_ID}/${name}" type="fixed"> <!-- continuous -->
+        <joint name="${ROBOT_ID}/${name}" type="continuous">
             <origin xyz="${origin_xyz}" rpy="${origin_rpy}"/>
             <parent link="${parent}"/>
@@ -35,4 +36,9 @@
             <axis xyz="${axis}" />
         </joint>
+        <xacro:if value="$(arg use_ros_control_for_base)">
+        <xacro:simple_transmission name="${ROBOT_ID}/${name}" interface="VelocityJointInterface"/>
+        </xacro:if>
+        <xacro:include filename="$(find mkmr_description)/urdf/mkmr/mkmr_wheels.gazebo.xacro"/>
+        <xacro:mkmr_wheels_gazebo/>
     </xacro:macro>
 </robot>
