Commit message: Update xacro files

File: mkmr_description/urdf/common/utils.urdf.xacro (robot description, xacro)
@@ -15,5 +15,5 @@
     <transmission name="${name}_trans">
       <type>transmission_interface/SimpleTransmission</type>
-      <joint name="${name}">
+      <joint name="${name}_joint">
         <hardwareInterface>hardware_interface/${interface}</hardwareInterface>
       </joint>

File: mkmr_description/urdf/mkmr.xacro (robot description, xacro)
@@ -21,6 +21,4 @@
     <xacro:mkmr_wheels parent="${ROBOT_ID}/base_link" name="front_right_wheel" origin_xyz="0.35336 -0.30481 -0.029122" origin_rpy="1.5708 0 -3.1416" axis="0 1 0"/>
     <xacro:mkmr_wheels parent="${ROBOT_ID}/base_link" name="rear_right_wheel" origin_xyz="0.18836 -0.30481 -0.031122" origin_rpy="-1.5708 0 0" axis="0 -1 0"/>
-    <!-- <xacro:mkmr_wheels parent="${ROBOT_ID}/base_link" name="left_wheel_joint" origin_xyz="0.18836 -0.30481 0.15588" origin_rpy="-1.5708 0 0" axis="0 -1 0"/> -->
-    <!-- <xacro:mkmr_wheels parent="${ROBOT_ID}/base_link" name="right_wheel_joint" origin_xyz="0.35336 -0.30481 -0.029122" origin_rpy="1.5708 0 -3.1416" axis="0 1 0"/> -->
     <!-- Laser -->
     <!-- <xacro:rplidar_a1 parent="${ROBOT_ID}/base_link" name="scan" origin_xyz="0.374625946277677 -0.494903544571783 0.0633776911630922" origin_rpy="0 0 3.14159265358979"/> -->

File: mkmr_description/urdf/mkmr/mkmr_wheels.urdf.xacro (robot description, xacro)
@@ -30,5 +30,5 @@
             </inertial>
         </link>
-        <joint name="${ROBOT_ID}/${name}" type="continuous">
+        <joint name="${ROBOT_ID}/${name}_joint" type="continuous">
             <origin xyz="${origin_xyz}" rpy="${origin_rpy}"/>
             <parent link="${parent}"/>
