Commit message: Update rplidar a1

File: mkmr_common/mkmr_description/urdf/sensors/rplidar_a1.gazebo.xacro (robot description, xacro)
@@ -7,5 +7,4 @@
     <gazebo reference="${ROBOT_ID}/${name}">
       <material>Gazebo/Black</material>
-        <!-- <xacro:unless value="${DUMMY}"> -->
         <sensor type="gpu_ray" name="${name}">
           <always_on>true</always_on>
@@ -16,5 +15,5 @@
             <scan>
               <horizontal>
-                <samples>811</samples>
+                <samples>720</samples>
                 <resolution>1</resolution>
                 <min_angle>${-1*M_PI}</min_angle>
@@ -23,5 +22,5 @@
             </scan>
             <range>
-              <min>0.05</min>
+              <min>0.15</min>
               <max>12.0</max>
               <resolution>0.01</resolution>
@@ -42,5 +41,4 @@
           </plugin>
         </sensor>
-      <!-- </xacro:unless> -->
     </gazebo>
   </xacro:macro>

File: mkmr_common/mkmr_description/urdf/sensors/rplidar_a1.urdf.xacro (robot description, xacro)
@@ -4,5 +4,5 @@
         <link name="${ROBOT_ID}/${name}">
             <visual>
-                <origin xyz="0 0 0" rpy="0 0 0"/>
+                <origin xyz="0 0 0" rpy="1.57 0 0"/>
                 <geometry>
                     <mesh filename="package://mkmr_description/meshes/${name}.STL" />
