Commit message: Fix rplidar stl visual yaw value

File: mkmr_common/mkmr_description/urdf/sensors/rplidar_a1.urdf.xacro (robot description, xacro)
@@ -4,5 +4,5 @@
         <link name="${ROBOT_ID}/${name}">
             <visual>
-                <origin xyz="0 0 0" rpy="1.57 0 0"/>
+                <origin xyz="0 0 0" rpy="1.57 0 -1.57"/>
                 <geometry>
                     <mesh filename="package://mkmr_description/meshes/${name}.STL" />
