Commit message: update wheel values

File: mkmr_common/mkmr_description/urdf/mkmr/mkmr_chasis.urdf.xacro (robot description, xacro)
@@ -38,7 +38,7 @@
     <link name="${ROBOT_ID}/front_left_wheel_link">
       <inertial>
-        <mass value="3"/>
+        <mass value="0.5"/>
         <origin xyz="0 0 0" rpy="0 ${M_PI/2} ${M_PI/2}"/>
-        <xacro:cylinder_inertia m="3" r="${wheel_radius}" h="${wheel_width}"/>
+        <xacro:cylinder_inertia m="0.5" r="${wheel_radius}" h="${wheel_width}"/>
       </inertial>
       <visual>
@@ -71,7 +71,7 @@
     <link name="${ROBOT_ID}/front_right_wheel_link">
       <inertial>
-        <mass value="3"/>
+        <mass value="0.5"/>
         <origin xyz="0 0 0" rpy="0 ${M_PI/2} ${M_PI/2}"/>
-        <xacro:cylinder_inertia m="3" r="${wheel_radius}" h="${wheel_width}"/>
+        <xacro:cylinder_inertia m="0.5" r="${wheel_radius}" h="${wheel_width}"/>
       </inertial>
       <visual>
@@ -104,7 +104,7 @@
     <link name="${ROBOT_ID}/rear_left_wheel_link">
       <inertial>
-        <mass value="3"/>
+        <mass value="0.5"/>
         <origin xyz="0 0 0" rpy="0 ${M_PI/2} ${M_PI/2}"/>
-        <xacro:cylinder_inertia m="3" r="${wheel_radius}" h="${wheel_width}"/>
+        <xacro:cylinder_inertia m="0.5" r="${wheel_radius}" h="${wheel_width}"/>
       </inertial>
       <visual>
@@ -137,7 +137,7 @@
     <link name="${ROBOT_ID}/rear_right_wheel_link">
       <inertial>
-        <mass value="3"/>
+        <mass value="0.5"/>
         <origin xyz="0 0 0" rpy="0 ${M_PI/2} ${M_PI/2}"/>
-        <xacro:cylinder_inertia m="3" r="${wheel_radius}" h="${wheel_width}"/>
+        <xacro:cylinder_inertia m="0.5" r="${wheel_radius}" h="${wheel_width}"/>
       </inertial>
       <visual>

File: mkmr_common/mkmr_description/urdf/mkmr/mkmr_wheels.gazebo.xacro (robot description, xacro)
@@ -12,7 +12,7 @@
         </visual>
         <kp>10000000.0</kp>
-        <kd>100.0</kd>
-        <mu1>1.0</mu1>
-        <mu2>1.0</mu2>
+        <kd>1.0</kd>
+        <mu1>200.0</mu1>
+        <mu2>200.0</mu2>
         <fdir1>1 1 1</fdir1>
         <minDepth>0.000</minDepth>

Commit message: Remove robot_id from joint_names

File: mkmr_common/mkmr_description/urdf/mkmr/mkmr_chasis.urdf.xacro (robot description, xacro)
@@ -57,5 +57,5 @@
       </collision>
     </link>
-    <joint name="${ROBOT_ID}/front_left_wheel_joint" type="continuous">
+    <joint name="front_left_wheel_joint" type="continuous">
       <origin xyz="${wheels_separation_x/2} ${wheels_separation_y/2} ${wheels_height}" rpy="0 0 0"/>
       <axis xyz="0 1 0"/>
@@ -66,5 +66,5 @@
     </joint>
     <xacro:if value="$(arg use_ros_control_for_base)">
-      <xacro:simple_transmission name="${ROBOT_ID}/front_left_wheel" interface="VelocityJointInterface"/>
+      <xacro:simple_transmission name="front_left_wheel" interface="VelocityJointInterface"/>
     </xacro:if>
     <!-- Right Wheel-->
@@ -90,5 +90,5 @@
       </collision>
     </link>
-    <joint name="${ROBOT_ID}/front_right_wheel_joint" type="continuous">
+    <joint name="front_right_wheel_joint" type="continuous">
       <origin xyz="${wheels_separation_x/2} ${(-1*wheels_separation_y)/2} ${wheels_height}" rpy="0 0 0"/>
       <axis xyz="0 1 0"/>
@@ -99,5 +99,5 @@
     </joint>
     <xacro:if value="$(arg use_ros_control_for_base)">
-      <xacro:simple_transmission name="${ROBOT_ID}/front_right_wheel" interface="VelocityJointInterface"/>
+      <xacro:simple_transmission name="front_right_wheel" interface="VelocityJointInterface"/>
     </xacro:if>
     <!-- Back Left Wheel-->
@@ -123,5 +123,5 @@
       </collision>
     </link>
-    <joint name="${ROBOT_ID}/rear_left_wheel_joint" type="continuous">
+    <joint name="rear_left_wheel_joint" type="continuous">
       <origin xyz="-${wheels_separation_x/2} ${wheels_separation_y/2} ${wheels_height}" rpy="0 0 0"/>
       <axis xyz="0 1 0"/>
@@ -132,5 +132,5 @@
     </joint>
     <xacro:if value="$(arg use_ros_control_for_base)">
-      <xacro:simple_transmission name="${ROBOT_ID}/rear_left_wheel" interface="VelocityJointInterface"/>
+      <xacro:simple_transmission name="rear_left_wheel" interface="VelocityJointInterface"/>
     </xacro:if>
     <!-- Back Right Wheel-->
@@ -156,5 +156,5 @@
       </collision>
     </link>
-    <joint name="${ROBOT_ID}/rear_right_wheel_joint" type="continuous">
+    <joint name="rear_right_wheel_joint" type="continuous">
       <origin xyz="-${wheels_separation_x/2} ${(-1*wheels_separation_y)/2} ${wheels_height}" rpy="0 0 0"/>
       <axis xyz="0 1 0"/>
@@ -165,5 +165,5 @@
     </joint>
     <xacro:if value="$(arg use_ros_control_for_base)">
-      <xacro:simple_transmission name="${ROBOT_ID}/rear_right_wheel" interface="VelocityJointInterface"/>
+      <xacro:simple_transmission name="rear_right_wheel" interface="VelocityJointInterface"/>
     </xacro:if>
     <xacro:include filename="$(find mkmr_description)/urdf/mkmr/mkmr_chasis.gazebo.xacro"/>

File: mkmr_common/mkmr_description/urdf/mkmr/mkmr_wheels.gazebo.xacro (robot description, xacro)
@@ -2,5 +2,5 @@
 <robot xmlns:xacro="http://ros.org/wiki/xacro">
     <xacro:macro name="mkmr_wheels_gazebo" params="name">
-      <gazebo reference="${ROBOT_ID}/${name}">
+      <gazebo reference="${name}">
         <visual>
           <material>
