Commit message: Add safety & warning zone

File: mkmr_common/mkmr_description/urdf/mkmr/mkmr_base.urdf.xacro (robot description, xacro)
@@ -2,15 +2,69 @@
 <robot xmlns:xacro="http://ros.org/wiki/xacro">
     <xacro:macro name="mkmr_base">
-        <!-- Base footprint -->
-        <link name="${ROBOT_ID}/base_footprint">
-        </link>
-        <!-- Base link -->
-        <link name="${ROBOT_ID}/base_link">
-        </link>
-        <joint name="${ROBOT_ID}/base_footprint_joint" type="fixed">
-            <origin xyz="0 0 0.04" rpy="0 0 0"/> <!-- drive wheel radius-->
-            <parent link="${ROBOT_ID}/base_footprint"/>
-            <child link="${ROBOT_ID}/base_link"/>
-        </joint>
+    <xacro:property name="robot_length_x" value="0.2"/>
+    <xacro:property name="robot_length_y" value="0.15"/>
+    <xacro:property name="runstop_dist" value="0.07"/>
+    <xacro:property name="normal_dist" value="${robot_length_x*2.6}"/>
+    <xacro:property name="normal_side_dist" value="${robot_length_y*1.5}"/>
+    <xacro:property name="slowdown_dist" value="${robot_length_x*2}"/>
+    <xacro:property name="slowdown_side_dist" value="${robot_length_y*1}"/>
+    <!-- Base footprint -->
+    <link name="${ROBOT_ID}/base_footprint">
+    </link>
+    <!-- Base link -->
+    <link name="${ROBOT_ID}/base_link">
+    </link>
+    <joint name="${ROBOT_ID}/base_footprint_joint" type="fixed">
+        <origin xyz="0 0 0.04" rpy="0 0 0"/> <!-- drive wheel radius-->
+        <parent link="${ROBOT_ID}/base_footprint"/>
+        <child link="${ROBOT_ID}/base_link"/>
+    </joint>
+    <link name="${ROBOT_ID}/base_cautious">
+        <visual>
+            <!-- <origin xyz="0.66875 0 0" rpy="0 0 0"/> -->
+            <origin xyz="0 0 0" rpy="0 0 0"/>
+            <geometry>
+                <!-- <box size ="1.3375 1.07 0.001"/> -->
+                <box size ="${normal_dist*2} ${(normal_side_dist+robot_length_x)*2} 0.001"/>
+            </geometry>
+            <material name="Yellow"/>
+        </visual>
+    </link>
+    <joint name="${ROBOT_ID}/base_cautious_joint" type="fixed">
+        <origin xyz="0 0 -0.115" rpy="0 0 0"/> <!-- drive wheel radius-->
+        <parent link="${ROBOT_ID}/base_link"/>
+        <child link="${ROBOT_ID}/base_cautious"/>
+    </joint>
+    <!-- Base footprint -->
+    <link name="${ROBOT_ID}/base_warning">
+        <visual>
+            <origin xyz="0 0 0" rpy="0 0 0"/>
+            <geometry>
+                <box size ="${slowdown_dist*2} ${(slowdown_side_dist+robot_length_y)*2} 0.002"/>
+            </geometry>
+            <material name="Orange"/>
+        </visual>
+    </link>
+    <joint name="${ROBOT_ID}/base_warning_joint" type="fixed">
+        <origin xyz="0 0 -0.115" rpy="0 0 0"/> <!-- drive wheel radius-->
+        <parent link="${ROBOT_ID}/base_link"/>
+        <child link="${ROBOT_ID}/base_warning"/>
+    </joint>
+    <link name="${ROBOT_ID}/base_safety">
+        <visual>
+            <!-- <origin xyz="0.1875 0 0" rpy="0 0 0"/> -->
+            <origin xyz="0 0 0" rpy="0 0 0"/>
+            <geometry>
+                <!-- <box size ="0.375 0.535 0.001"/> -->
+                <box size ="${runstop_dist*2+robot_length_x*2} ${runstop_dist*2+robot_length_y*2} 0.003"/>
+            </geometry>
+            <material name="Red"/>
+        </visual>
+    </link>
+    <joint name="${ROBOT_ID}/base_safety_joint" type="fixed">
+        <origin xyz="0 0 -0.115" rpy="0 0 0"/> <!-- drive wheel radius-->
+        <parent link="${ROBOT_ID}/base_link"/>
+        <child link="${ROBOT_ID}/base_safety"/>
+    </joint>
     <xacro:include filename="$(find mkmr_description)/urdf/mkmr/mkmr_chasis.urdf.xacro"/>
     <xacro:chasis parent="${ROBOT_ID}/base_link"/>

Commit message: Update safety & warning zones

File: mkmr_common/mkmr_description/urdf/mkmr/mkmr_base.urdf.xacro (robot description, xacro)
@@ -4,9 +4,9 @@
     <xacro:property name="robot_length_x" value="0.2"/>
     <xacro:property name="robot_length_y" value="0.15"/>
-    <xacro:property name="runstop_dist" value="0.07"/>
-    <xacro:property name="normal_dist" value="${robot_length_x*2.6}"/>
-    <xacro:property name="normal_side_dist" value="${robot_length_y*1.5}"/>
-    <xacro:property name="slowdown_dist" value="${robot_length_x*2}"/>
-    <xacro:property name="slowdown_side_dist" value="${robot_length_y*1}"/>
+    <xacro:property name="safety_offset" value="0.1"/>
+    <xacro:property name="normal_dist" value="${robot_length_x*4}"/>
+    <xacro:property name="normal_side_dist" value="${robot_length_y*2.5}"/>
+    <xacro:property name="slow_dist" value="${robot_length_x*3}"/>
+    <xacro:property name="slow_side_dist" value="${robot_length_y*1.5}"/>
     <!-- Base footprint -->
     <link name="${ROBOT_ID}/base_footprint">
@@ -28,5 +28,5 @@
                 <box size ="${normal_dist*2} ${(normal_side_dist+robot_length_x)*2} 0.001"/>
             </geometry>
-            <material name="Yellow"/>
+            <material name="Light_Blue"/>
         </visual>
     </link>
@@ -41,7 +41,7 @@
             <origin xyz="0 0 0" rpy="0 0 0"/>
             <geometry>
-                <box size ="${slowdown_dist*2} ${(slowdown_side_dist+robot_length_y)*2} 0.002"/>
+                <box size ="${slow_dist*2} ${(slow_side_dist+robot_length_y)*2} 0.002"/>
             </geometry>
-            <material name="Orange"/>
+            <material name="Yellow"/>
         </visual>
     </link>
@@ -57,5 +57,5 @@
             <geometry>
                 <!-- <box size ="0.375 0.535 0.001"/> -->
-                <box size ="${runstop_dist*2+robot_length_x*2} ${runstop_dist*2+robot_length_y*2} 0.003"/>
+                <box size ="${safety_offset*2+robot_length_x*2} ${safety_offset*2+robot_length_y*2} 0.003"/>
             </geometry>
             <material name="Red"/>

Commit message: update zones in urdf

File: mkmr_common/mkmr_description/urdf/mkmr/mkmr_base.urdf.xacro (robot description, xacro)
@@ -22,8 +22,6 @@
     <link name="${ROBOT_ID}/base_cautious">
         <visual>
-            <!-- <origin xyz="0.66875 0 0" rpy="0 0 0"/> -->
-            <origin xyz="0 0 0" rpy="0 0 0"/>
+            <origin xyz="0 0 -0.02" rpy="0 0 0"/>
             <geometry>
-                <!-- <box size ="1.3375 1.07 0.001"/> -->
                 <box size ="${normal_dist*2} ${(normal_side_dist+robot_length_x)*2} 0.001"/>
             </geometry>
@@ -32,12 +30,11 @@
     </link>
     <joint name="${ROBOT_ID}/base_cautious_joint" type="fixed">
-        <origin xyz="0 0 -0.115" rpy="0 0 0"/> <!-- drive wheel radius-->
+        <origin xyz="0 0 0.0" rpy="0 0 0"/>
         <parent link="${ROBOT_ID}/base_link"/>
         <child link="${ROBOT_ID}/base_cautious"/>
     </joint>
-    <!-- Base footprint -->
     <link name="${ROBOT_ID}/base_warning">
         <visual>
-            <origin xyz="0 0 0" rpy="0 0 0"/>
+            <origin xyz="0 0 -0.01" rpy="0 0 0"/>
             <geometry>
                 <box size ="${slow_dist*2} ${(slow_side_dist+robot_length_y)*2} 0.002"/>
@@ -47,5 +44,5 @@
     </link>
     <joint name="${ROBOT_ID}/base_warning_joint" type="fixed">
-        <origin xyz="0 0 -0.115" rpy="0 0 0"/> <!-- drive wheel radius-->
+        <origin xyz="0 0 0.0" rpy="0 0 0"/>
         <parent link="${ROBOT_ID}/base_link"/>
         <child link="${ROBOT_ID}/base_warning"/>
@@ -53,8 +50,6 @@
     <link name="${ROBOT_ID}/base_safety">
         <visual>
-            <!-- <origin xyz="0.1875 0 0" rpy="0 0 0"/> -->
             <origin xyz="0 0 0" rpy="0 0 0"/>
             <geometry>
-                <!-- <box size ="0.375 0.535 0.001"/> -->
                 <box size ="${safety_offset*2+robot_length_x*2} ${safety_offset*2+robot_length_y*2} 0.003"/>
             </geometry>
@@ -63,5 +58,5 @@
     </link>
     <joint name="${ROBOT_ID}/base_safety_joint" type="fixed">
-        <origin xyz="0 0 -0.115" rpy="0 0 0"/> <!-- drive wheel radius-->
+        <origin xyz="0 0 0.0" rpy="0 0 0"/>
         <parent link="${ROBOT_ID}/base_link"/>
         <child link="${ROBOT_ID}/base_safety"/>

Commit message: fix zones origin z offset

File: mkmr_common/mkmr_description/urdf/mkmr/mkmr_base.urdf.xacro (robot description, xacro)
@@ -22,5 +22,5 @@
     <link name="${ROBOT_ID}/base_cautious">
         <visual>
-            <origin xyz="0 0 -0.02" rpy="0 0 0"/>
+            <origin xyz="0 0 -0.04" rpy="0 0 0"/>
             <geometry>
                 <box size ="${normal_dist*2} ${(normal_side_dist+robot_length_x)*2} 0.001"/>
@@ -36,5 +36,5 @@
     <link name="${ROBOT_ID}/base_warning">
         <visual>
-            <origin xyz="0 0 -0.01" rpy="0 0 0"/>
+            <origin xyz="0 0 -0.04" rpy="0 0 0"/>
             <geometry>
                 <box size ="${slow_dist*2} ${(slow_side_dist+robot_length_y)*2} 0.002"/>
@@ -50,5 +50,5 @@
     <link name="${ROBOT_ID}/base_safety">
         <visual>
-            <origin xyz="0 0 0" rpy="0 0 0"/>
+            <origin xyz="0 0 -0.04" rpy="0 0 0"/>
             <geometry>
                 <box size ="${safety_offset*2+robot_length_x*2} ${safety_offset*2+robot_length_y*2} 0.003"/>

Commit message: Create mkmr_p_prod pkg

File: mkmr_common/mkmr_description/urdf/mkmr/mkmr_base.urdf.xacro (robot description, xacro)
@@ -5,8 +5,16 @@
     <xacro:property name="robot_length_y" value="0.15"/>
     <xacro:property name="safety_offset" value="0.1"/>
-    <xacro:property name="normal_dist" value="${robot_length_x*4}"/>
-    <xacro:property name="normal_side_dist" value="${robot_length_y*2.5}"/>
-    <xacro:property name="slow_dist" value="${robot_length_x*3}"/>
-    <xacro:property name="slow_side_dist" value="${robot_length_y*1.5}"/>
+    <xacro:if value="${IS_SIM}">
+        <xacro:property name="normal_dist" value="${robot_length_x*4}"/>
+        <xacro:property name="normal_side_dist" value="${robot_length_y*2.5}"/>
+        <xacro:property name="slow_dist" value="${robot_length_x*3}"/>
+        <xacro:property name="slow_side_dist" value="${robot_length_y*1.5}"/>
+    </xacro:if>
+    <xacro:unless value="${IS_SIM}">
+        <xacro:property name="normal_dist" value="${robot_length_x*2}"/>
+        <xacro:property name="normal_side_dist" value="${robot_length_y*1.5}"/>
+        <xacro:property name="slow_dist" value="${robot_length_x*1.5}"/>
+        <xacro:property name="slow_side_dist" value="${robot_length_y*0.5}"/>
+    </xacro:unless>
     <!-- Base footprint -->
     <link name="${ROBOT_ID}/base_footprint">

Commit message: Update urdf zones

File: mkmr_common/mkmr_description/urdf/mkmr/mkmr_base.urdf.xacro (robot description, xacro)
@@ -4,6 +4,6 @@
     <xacro:property name="robot_length_x" value="0.2"/>
     <xacro:property name="robot_length_y" value="0.15"/>
-    <xacro:property name="safety_offset" value="0.1"/>
     <xacro:if value="${IS_SIM}">
+        <xacro:property name="safety_offset" value="0.1"/>
         <xacro:property name="normal_dist" value="${robot_length_x*4}"/>
         <xacro:property name="normal_side_dist" value="${robot_length_y*2.5}"/>
@@ -12,8 +12,9 @@
     </xacro:if>
     <xacro:unless value="${IS_SIM}">
-        <xacro:property name="normal_dist" value="${robot_length_x*2}"/>
+        <xacro:property name="safety_offset" value="0.04"/>
+        <xacro:property name="normal_dist" value="${robot_length_x*2.5}"/>
         <xacro:property name="normal_side_dist" value="${robot_length_y*1.5}"/>
-        <xacro:property name="slow_dist" value="${robot_length_x*1.5}"/>
-        <xacro:property name="slow_side_dist" value="${robot_length_y*0.5}"/>
+        <xacro:property name="slow_dist" value="${robot_length_x*1.75}"/>
+        <xacro:property name="slow_side_dist" value="${robot_length_y*1.0}"/>
     </xacro:unless>
     <!-- Base footprint -->
