Commit message: Update urdf stl  files

File: mkmr_common/mkmr_description/urdf/mkmr.xacro (robot description, xacro)
@@ -12,13 +12,7 @@
     <xacro:include filename="$(find mkmr_description)/urdf/common/plugins.gazebo.xacro"/>
     <xacro:include filename="$(find mkmr_description)/urdf/mkmr/mkmr_base.urdf.xacro"/>
-    <xacro:include filename="$(find mkmr_description)/urdf/mkmr/mkmr_wheels.urdf.xacro"/>
     <xacro:include filename="$(find mkmr_description)/urdf/sensors/rplidar_a1.urdf.xacro"/>
     <!-- Robot Base-->
     <xacro:mkmr_base/>
-     <!-- Wheels -->
-    <xacro:mkmr_wheels parent="${ROBOT_ID}/base_link" name="front_left_wheel" origin_xyz="0.35336 -0.30481 0.15788" origin_rpy="1.5708 0 -3.1416" axis="0 1 0"/>
-    <xacro:mkmr_wheels parent="${ROBOT_ID}/base_link" name="rear_left_wheel" origin_xyz="0.18836 -0.30481 0.15588" origin_rpy="-1.5708 0 0" axis="0 -1 0"/>
-    <xacro:mkmr_wheels parent="${ROBOT_ID}/base_link" name="front_right_wheel" origin_xyz="0.35336 -0.30481 -0.029122" origin_rpy="1.5708 0 -3.1416" axis="0 1 0"/>
-    <xacro:mkmr_wheels parent="${ROBOT_ID}/base_link" name="rear_right_wheel" origin_xyz="0.18836 -0.30481 -0.031122" origin_rpy="-1.5708 0 0" axis="0 -1 0"/>
     <!-- Laser -->
     <!-- <xacro:rplidar_a1 parent="${ROBOT_ID}/base_link" name="scan" origin_xyz="0.374625946277677 -0.494903544571783 0.0633776911630922" origin_rpy="0 0 3.14159265358979"/> -->

File: mkmr_common/mkmr_description/urdf/mkmr/mkmr_base.urdf.xacro (robot description, xacro)
@@ -1,49 +1,52 @@
 <?xml version="1.0"?>
-<robot xmlns:xacro="http://ros.org/wiki/xacro" name="mkmr" >
+<robot xmlns:xacro="http://ros.org/wiki/xacro">
     <xacro:macro name="mkmr_base">
         <!-- Base footprint -->
         <link name="${ROBOT_ID}/base_footprint">
-            <visual>
-                <origin xyz="0.28 0 0" rpy="0 0 0"/>
-                <geometry>
-                    <box size ="0.3 0.4 0.001"/>
-                </geometry>
-                <material name="Orange"/>
-            </visual>
         </link>
         <!-- Base link -->
         <link name="${ROBOT_ID}/base_link">
+        </link>
+        <joint name="${ROBOT_ID}/base_footprint_joint" type="fixed">
+            <origin xyz="0 0 0.04" rpy="0 0 0"/> <!-- drive wheel radius-->
+            <parent link="${ROBOT_ID}/base_footprint"/>
+            <child link="${ROBOT_ID}/base_link"/>
+        </joint>
+    <xacro:include filename="$(find mkmr_description)/urdf/mkmr/mkmr_chasis.urdf.xacro"/>
+    <xacro:chasis parent="${ROBOT_ID}/base_link"/>
+        <!-- fMotorBracket -->
+        <!-- <link name="${ROBOT_ID}/fMotorBracket">
             <visual>
                 <origin xyz="0 0 0" rpy="0 0 0"/>
                 <geometry>
-                    <mesh filename="package://mkmr_description/meshes/base_link.STL" />
+                    <mesh filename="package://mkmr_description/meshes/fMotorBracket.STL" />
                 </geometry>
                 <material name="Black"/>
             </visual>
             <collision>
-                <origin xyz="0 0 0.01" rpy="0 0 0"/><!-- 1 cm above for wheel trick -->
+                <origin xyz="0 0 0" rpy="0 0 0"/>
                 <geometry>
-                    <mesh filename="package://mkmr_description/meshes/base_link.STL" />
+                    <mesh filename="package://mkmr_description/meshes/fMotorBracket.STL" />
                 </geometry>
             </collision>
             <inertial>
-                <origin xyz="0.277007577638953 -0.338806344571783 0.0633776923791692"/>
-                <mass value="0.1"/>
+                <origin xyz="-0.0610000000000015 -0.0674547790002785 -0.0116887463358963"/>
+                <mass value="0.2"/>
                 <inertia
-                    ixx="0.000191833350350532"
-                    ixy="3.81016043819389E-18"
-                    ixz="1.43353501127755E-11"
-                    iyy="0.000732589595457571"
-                    iyz="2.42104727054767E-16"
-                    izz="0.000540911588861397" />
+                    ixx="3.51055038644331E-06"
+                    ixy="-6.12729326621837E-19"
+                    ixz="8.524624284462E-17"
+                    iyy="3.95634077909559E-06"
+                    iyz="1.11448332781975E-19"
+                    izz="3.62492890882267E-06" />
             </inertial>
         </link>
-        <joint name="${ROBOT_ID}/base_footprint_joint" type="fixed">
-            <origin xyz="-0.274  -0.062   -0.275" rpy="-1.57 0 0"/> <!-- drive wheel radius-->
-            <parent link="${ROBOT_ID}/base_footprint"/>
-            <child link="${ROBOT_ID}/base_link"/>
-        </joint>
+        <joint name="${ROBOT_ID}/fMotorBracket_joint" type="fixed">
+            <origin xyz="0.0345000000000004 0 -0.0609999999999998" rpy="1.5707963267949 1.5707963267949 0"/>
+            <parent link="${ROBOT_ID}/base_link"/>
+            <child link="${ROBOT_ID}/fMotorBracket"/>
+        </joint> -->
         <!-- fMotor -->
-        <link name="${ROBOT_ID}/fMotor">
+        <!-- <link name="${ROBOT_ID}/fMotor">
             <visual>
                 <origin xyz="0 0 0" rpy="0 0 0"/>
@@ -60,22 +63,22 @@
             </collision>
             <inertial>
-                <origin xyz="-2.35922392732846E-16 -0.0329974549151947 -0.02859664503564"/>
-                <mass value="0.8"/>
+                <origin xyz="0.0012598162449621 0.0824999999999999 -0.079"/>
+                <mass value="0.2"/>
                 <inertia
-                    ixx="3.18777376766978E-05"
-                    ixy="2.71802092193263E-07"
-                    ixz="8.53012918247537E-17"
-                    iyy="5.51232387338385E-05"
-                    iyz="1.0709267346185E-19"
-                    izz="5.4667129576926E-05" />
+                    ixx="5.17259698645822E-05"
+                    ixy="-5.07691498136368E-23"
+                    ixz="-7.9467054546941E-20"
+                    iyy="5.18506671512217E-05"
+                    iyz="2.71802092193946E-07"
+                    izz="2.83766813003582E-05" />
             </inertial>
         </link>
         <joint name="${ROBOT_ID}/fMotor_joint" type="fixed">
-            <origin xyz="0.30386 -0.34031 0.063378" rpy="1.5708 1.5708 0"/>
-            <parent link="${ROBOT_ID}/base_link"/>
+            <origin xyz="0.0179999999999999 -0.15 -0.0285000000000011" rpy="0 1.5707963267949 0"/>
+            <parent link="${ROBOT_ID}/fMotorBracket"/>
             <child link="${ROBOT_ID}/fMotor"/>
-        </joint>
+        </joint> -->
         <!-- fDrivers -->
-        <link name="${ROBOT_ID}/fDrivers">
+        <!-- <link name="${ROBOT_ID}/fDrivers">
             <visual>
                 <origin xyz="0 0 0" rpy="0 0 0"/>
@@ -107,5 +110,5 @@
             <parent link="${ROBOT_ID}/base_link"/>
             <child link="${ROBOT_ID}/fDrivers"/>
-        </joint>
+        </joint> -->
     </xacro:macro>
 </robot>

File: mkmr_common/mkmr_description/urdf/mkmr/mkmr_wheels.gazebo.xacro (robot description, xacro)
@@ -1,5 +1,5 @@
 <?xml version="1.0"?>
 <robot xmlns:xacro="http://ros.org/wiki/xacro">
-    <xacro:macro name="mkmr_wheels_gazebo">
+    <xacro:macro name="mkmr_wheels_gazebo" params="name">
       <gazebo reference="${ROBOT_ID}/${name}">
         <visual>

File: mkmr_common/mkmr_description/urdf/sensors/rplidar_a1.urdf.xacro (robot description, xacro)
@@ -1,4 +1,4 @@
 <?xml version="1.0"?>
-<robot xmlns:xacro="http://ros.org/wiki/xacro" name="mkmr" >
+<robot xmlns:xacro="http://ros.org/wiki/xacro">
     <xacro:macro name="rplidar_a1" params="parent name origin_xyz origin_rpy">
         <link name="${ROBOT_ID}/${name}">

Commit message: Update urdf files

File: mkmr_common/mkmr_description/urdf/mkmr.xacro (robot description, xacro)
@@ -12,7 +12,10 @@
     <xacro:include filename="$(find mkmr_description)/urdf/common/plugins.gazebo.xacro"/>
     <xacro:include filename="$(find mkmr_description)/urdf/mkmr/mkmr_base.urdf.xacro"/>
+    <xacro:include filename="$(find mkmr_description)/urdf/mkmr/mkmr_fixed.urdf.xacro"/>
     <xacro:include filename="$(find mkmr_description)/urdf/sensors/rplidar_a1.urdf.xacro"/>
     <!-- Robot Base-->
     <xacro:mkmr_base/>
+    <!-- Robot Fixed-->
+    <xacro:mkmr_fixed/>
     <!-- Laser -->
     <!-- <xacro:rplidar_a1 parent="${ROBOT_ID}/base_link" name="scan" origin_xyz="0.374625946277677 -0.494903544571783 0.0633776911630922" origin_rpy="0 0 3.14159265358979"/> -->

File: mkmr_common/mkmr_description/urdf/mkmr/mkmr_base.urdf.xacro (robot description, xacro)
@@ -15,100 +15,4 @@
     <xacro:include filename="$(find mkmr_description)/urdf/mkmr/mkmr_chasis.urdf.xacro"/>
     <xacro:chasis parent="${ROBOT_ID}/base_link"/>
-        <!-- fMotorBracket -->
-        <!-- <link name="${ROBOT_ID}/fMotorBracket">
-            <visual>
-                <origin xyz="0 0 0" rpy="0 0 0"/>
-                <geometry>
-                    <mesh filename="package://mkmr_description/meshes/fMotorBracket.STL" />
-                </geometry>
-                <material name="Black"/>
-            </visual>
-            <collision>
-                <origin xyz="0 0 0" rpy="0 0 0"/>
-                <geometry>
-                    <mesh filename="package://mkmr_description/meshes/fMotorBracket.STL" />
-                </geometry>
-            </collision>
-            <inertial>
-                <origin xyz="-0.0610000000000015 -0.0674547790002785 -0.0116887463358963"/>
-                <mass value="0.2"/>
-                <inertia
-                    ixx="3.51055038644331E-06"
-                    ixy="-6.12729326621837E-19"
-                    ixz="8.524624284462E-17"
-                    iyy="3.95634077909559E-06"
-                    iyz="1.11448332781975E-19"
-                    izz="3.62492890882267E-06" />
-            </inertial>
-        </link>
-        <joint name="${ROBOT_ID}/fMotorBracket_joint" type="fixed">
-            <origin xyz="0.0345000000000004 0 -0.0609999999999998" rpy="1.5707963267949 1.5707963267949 0"/>
-            <parent link="${ROBOT_ID}/base_link"/>
-            <child link="${ROBOT_ID}/fMotorBracket"/>
-        </joint> -->
-        <!-- fMotor -->
-        <!-- <link name="${ROBOT_ID}/fMotor">
-            <visual>
-                <origin xyz="0 0 0" rpy="0 0 0"/>
-                <geometry>
-                    <mesh filename="package://mkmr_description/meshes/fMotor.STL" />
-                </geometry>
-                <material name="Black"/>
-            </visual>
-            <collision>
-                <origin xyz="0 0 0" rpy="0 0 0"/>
-                <geometry>
-                    <mesh filename="package://mkmr_description/meshes/fMotor.STL" />
-                </geometry>
-            </collision>
-            <inertial>
-                <origin xyz="0.0012598162449621 0.0824999999999999 -0.079"/>
-                <mass value="0.2"/>
-                <inertia
-                    ixx="5.17259698645822E-05"
-                    ixy="-5.07691498136368E-23"
-                    ixz="-7.9467054546941E-20"
-                    iyy="5.18506671512217E-05"
-                    iyz="2.71802092193946E-07"
-                    izz="2.83766813003582E-05" />
-            </inertial>
-        </link>
-        <joint name="${ROBOT_ID}/fMotor_joint" type="fixed">
-            <origin xyz="0.0179999999999999 -0.15 -0.0285000000000011" rpy="0 1.5707963267949 0"/>
-            <parent link="${ROBOT_ID}/fMotorBracket"/>
-            <child link="${ROBOT_ID}/fMotor"/>
-        </joint> -->
-        <!-- fDrivers -->
-        <!-- <link name="${ROBOT_ID}/fDrivers">
-            <visual>
-                <origin xyz="0 0 0" rpy="0 0 0"/>
-                <geometry>
-                    <mesh filename="package://mkmr_description/meshes/fDrivers.STL" />
-                </geometry>
-                <material name="Black"/>
-            </visual>
-            <collision>
-                <origin xyz="0 0 0" rpy="0 0 0"/>
-                <geometry>
-                    <mesh filename="package://mkmr_description/meshes/fDrivers.STL" />
-                </geometry>
-            </collision>
-            <inertial>
-                <origin xyz="-0.00660140608489862 0.0452390915749958 -0.00380039164943846"/>
-                <mass value="0.3"/>
-                <inertia
-                    ixx="9.00028132290921E-06"
-                    ixy="1.23322543868992E-07"
-                    ixz="1.33828527421449E-07"
-                    iyy="2.17066983097978E-05"
-                    iyz="7.70745731959558E-07"
-                    izz="2.83837538531001E-05" />
-            </inertial>
-        </link>
-        <joint name="${ROBOT_ID}/fDrivers_joint" type="fixed">
-            <origin xyz="0.26391 -0.33566 0.1011" rpy="-1.5708 0 -3.1416"/>
-            <parent link="${ROBOT_ID}/base_link"/>
-            <child link="${ROBOT_ID}/fDrivers"/>
-        </joint> -->
     </xacro:macro>
 </robot>

Commit message: Fix lidar frame values

File: mkmr_common/mkmr_description/urdf/mkmr.xacro (robot description, xacro)
@@ -22,5 +22,5 @@
     <xacro:rplidar_a1 parent="${ROBOT_ID}/base_link"
                         name="scan"
-                        origin_xyz="0.07 0 0.124"
+                        origin_xyz="0.07 0 0.13"
                         origin_rpy="0 0 0"/>
 </robot>

File: mkmr_common/mkmr_description/urdf/mkmr/mkmr_fixed.urdf.xacro (robot description, xacro)
@@ -190,5 +190,5 @@
         </link>
         <joint name="${ROBOT_ID}/fPC_joint" type="fixed">
-            <origin xyz="0.02413 -0.0322100000000002 0" rpy="3.14159265358979 1.5707963267949 0"/>
+            <origin xyz="0.02413 -0.0322100000000002 0.01" rpy="3.14159265358979 1.5707963267949 0"/>
             <parent link="${ROBOT_ID}/fBase"/>
             <child link="${ROBOT_ID}/fPC"/>
